File: measurementcircuit/measurementcircuit.kicad_sch (KiCad schematic)
At the start: 81 parts, among them J1 Conn_01x02, J10 Conn_01x02, J11 Conn_01x02, J12 Conn_01x02, J13 250-108/000-006, J15 Conn_01x02, J16 Conn_01x02, J17 250-116/000-012, J18 2604-3102, J19 2604-3102, J2 Conn_01x02, J20 2604-3102, J21 Conn_01x02, J22 Conn_01x02, J23 Conn_01x02, J24 Conn_01x02, J25 Conn_01x02, J26 Conn_01x02, J27 Conn_01x02, J28 Conn_01x02, J29 Conn_01x02, J3 2604-3102, J30 Conn_01x02, J31 Conn_01x02, J32 Conn_01x02, J33 Conn_01x02, J34 Conn_01x02, J35 Conn_01x02, J36 Conn_01x02, J37 Conn_01x02, J38 Conn_01x02, J39 Conn_01x02, J4 2604-3102, J40 Conn_01x02, J41 Conn_01x02, J42 Conn_01x02, J5 2604-3102, J6 2604-3102, J7 2604-3102, J8 Conn_01x02, J9 Conn_01x02

Commit message: Redesign Work - Symbols, Schematic Overhaul
Parts:
- removed J13: 250-108/000-006, WAGO_250-108/000-006_connector_BLUE.pretty:CONN8_250-108&slash_000-006_WAG, symbol WAGO_Connectors:250-108_000-006
- removed J17: 250-116/000-012, Senior_Design:CONN16_250-116&slash_000-012_WAG, symbol CONN16:250-116_000-012
- added C10, C9: C3216X7R1E475K160AC, CAP_3216_TDK, symbol Bulk_Cap_2025-12-21_04-50-52:C3216X7R1E475K160AC
- added C11, C12, C13, C14, C15, C16, C18: 10pF, Capacitor_SMD:C_0805_2012Metric, symbol Device:C
- added C17: 10pF, 10pF_Capacitor_Custom:C_Disc_Radial_P5.90mm_W4.3mm_L11.4mm_Placeholder, symbol Device:C
- added J13, J50, J55, J61, J66, J71, J76, J81: 2604-3102, Wago - 2604-3302_2_pole_connector:CONN2_2604-3302_WAG, symbol CONN2:2604-3102
- added J14, J43: DILB28P-223TLF, DILB28P-223TLF:AMPHENOL_DILB28P-223TLF, symbol DIP_Socket_DILB28P-223TLF:DILB28P-223TLF
- added J17, J47, J48, J49, J51, J52, J53, J54, J56, J57, J58, J59, J62, J63, J64, J65, J67, J68, J69, J70, J72, J73, J74, J75, J77, J78, J79, J80, J82, J83, J84: Conn_01x02, Connector_PinHeader_2.54mm:PinHeader_1x02_P2.54mm_Vertical, symbol Connector_Generic:Conn_01x02
- added J44: 2601-1102, CONN2_2601-1102_WAG, symbol 2_Pole_Terminal_Block_2025-12-21_05-29-27:2601-1102
- added J45, J46, J60: 2601-1108, CONN8_2601-1108_WAG, symbol 8_Pole_Terminal_Block_2025-12-21_05-24-59:2601-1108
- added L10, L11, L12, L13, L14, L15, L16, L9: 56μH, Inductor_SMD:L_0805_2012Metric, symbol Device:L
- added R25, R28, R31, R34, R37, R40, R43, R46: 10 Ohm, Resistor_THT:R_Axial_Power_L38.0mm_W9.0mm_P40.64mm, symbol Device:R
- added R26, R29, R32, R35, R38, R41, R44, R47: 50 Ohm, Resistor_THT:R_Axial_Power_L20.0mm_W6.4mm_P25.40mm, symbol Device:R
- added R27, R30, R33, R36, R39, R42, R45, R48: 500 Ohm, Resistor_THT:R_Axial_DIN0309_L9.0mm_D3.2mm_P5.08mm_Vertical, symbol Device:R
- C1: footprint Capacitor_SMD:C_0805_2012Metric -> 10pF_Capacitor_Custom:C_Disc_Radial_P5.90mm_W4.3mm_L11.4mm_Placeholder
Connections:
- net GND: now also C11.2, C12.2, C13.2, C14.2, C15.2, C16.2, C17.2, C18.2, J13.3 (2_1), J13.4 (2_2), J50.3 (2_1), J50.4 (2_2), J55.3 (2_1), J55.4 (2_2), J61.3 (2_1), J61.4 (2_2), J66.3 (2_1), J66.4 (2_2), J71.3 (2_1), J71.4 (2_2), J76.3 (2_1), J76.4 (2_2), J81.3 (2_1), J81.4 (2_2)
- net at C8.1, L8.2, R22.2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: now also J43.11
- net at C6.1, L6.2, R16.2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: now also J43.09
- net at J16.1 (Pin_1), J20.1 (1_1), J20.2 (1_2)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: now also J14.11
- net at J10.2 (Pin_2), J25.1 (Pin_1), J26.1 (Pin_1)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: now also J14.06
- net at C1.1, J4.1 (1_1), J4.2 (1_2)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: now also J14.05, J43.05
- net at C4.1, L4.2, R10.2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: now also J43.07; no longer J11.2 (Pin_2), J6.1 (1_1), J6.2 (1_2)
- net at J1.1 (Pin_1), J2.1 (Pin_1), J21.1 (Pin_1)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: now also J14.04
- net at C3.1, L3.2, R7.2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: now also J43.06
- net at J10.1 (Pin_1), J28.1 (Pin_1), J29.1 (Pin_1)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: now also J11.2 (Pin_2), J6.1 (1_1), J6.2 (1_2), J14.07
- net at C2.1, L1.2, R1.2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: now also J43.04
- net at L5.1: now also J46.7 (4_1), J46.8 (4_2)
- net at C5.1, L5.2, R13.2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: now also J43.08
- net at J11.1 (Pin_1), J12.2 (Pin_2), J31.1 (Pin_1)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: now also J14.08
- net at J12.1 (Pin_1), J15.2 (Pin_2), J18.1 (1_1)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: now also J14.09
- net at J15.1 (Pin_1), J16.2 (Pin_2), J19.1 (1_1)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: now also J14.10
- net at C7.1, L7.2, R19.2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: now also J43.10
- net at L1.1: now also J46.15 (8_1), J46.16 (8_2)
- net at L4.1: now also J46.10 (5_2), J46.9 (5_1)
- net at L7.1: now also J46.3 (2_1), J46.4 (2_2)
- net at L2.1: now also J46.13 (7_1), J46.14 (7_2)
- net at L8.1: now also J46.1 (1_1), J46.2 (1_2)
- net at L3.1: now also J46.11 (6_1), J46.12 (6_2)
- net at L6.1: now also J46.5 (3_1), J46.6 (3_2)
- new net: J14.22, J65.2 (Pin_2), J66.1 (1_1), J66.2 (1_2), J67.1 (Pin_1), J68.1 (Pin_1), J69.1 (Pin_1), J70.1 (Pin_1)
- new net: J67.2 (Pin_2), R37.1
- new net: J14.25, J49.2 (Pin_2), J50.1 (1_1), J50.2 (1_2), J51.1 (Pin_1), J52.1 (Pin_1), J53.1 (Pin_1), J54.1 (Pin_1)
- new net: J14.24, J54.2 (Pin_2), J55.1 (1_1), J55.2 (1_2), J56.1 (Pin_1), J57.1 (Pin_1), J58.1 (Pin_1), J59.1 (Pin_1)
- new net: J14.19, J80.2 (Pin_2), J81.1 (1_1), J81.2 (1_2), J82.1 (Pin_1), J83.1 (Pin_1), J84.1 (Pin_1)
- new net: J83.2 (Pin_2), R47.1
- new net: J13.1 (1_1), J13.2 (1_2), J14.26, J17.1 (Pin_1), J47.1 (Pin_1), J48.1 (Pin_1), J49.1 (Pin_1)
- new net: J17.2 (Pin_2), R25.1
- new net: J60.10 (5_2), J60.9 (5_1), L13.1
- new net: C15.1, J43.22, L13.2, R37.2, R38.2, R39.2
- new net: J14.21, J70.2 (Pin_2), J71.1 (1_1), J71.2 (1_2), J72.1 (Pin_1), J73.1 (Pin_1), J74.1 (Pin_1), J75.1 (Pin_1)
- new net: J72.2 (Pin_2), R40.1
- new net: J74.2 (Pin_2), R42.1
- new net: C16.1, J43.21, L14.2, R40.2, R41.2, R42.2
- new net: J14.20, J75.2 (Pin_2), J76.1 (1_1), J76.2 (1_2), J77.1 (Pin_1), J78.1 (Pin_1), J79.1 (Pin_1), J80.1 (Pin_1)
- new net: J78.2 (Pin_2), R44.1
- new net: C18.1, J43.19, L16.2, R46.2, R47.2, R48.2
- new net: J58.2 (Pin_2), R33.1
- new net: J51.2 (Pin_2), R28.1
- new net: C12.1, J43.25, L10.2, R28.2, R29.2, R30.2
- new net: J82.2 (Pin_2), R46.1
- new net: J53.2 (Pin_2), R30.1
- new net: J60.13 (7_1), J60.14 (7_2), L15.1
- new net: C17.1, J43.20, L15.2, R43.2, R44.2, R45.2
- new net: J60.1 (1_1), J60.2 (1_2), L9.1
- new net: J60.11 (6_1), J60.12 (6_2), L14.1
- new net: J60.15 (8_1), J60.16 (8_2), L16.1
- new net: J60.3 (2_1), J60.4 (2_2), L10.1
- new net: J60.5 (3_1), J60.6 (3_2), L11.1
- new net: J60.7 (4_1), J60.8 (4_2), L12.1
- new net: J14.23, J59.2 (Pin_2), J61.1 (1_1), J61.2 (1_2), J62.1 (Pin_1), J63.1 (Pin_1), J64.1 (Pin_1), J65.1 (Pin_1)
- new net: J64.2 (Pin_2), R36.1
- new net: C13.1, J43.24, L11.2, R31.2, R32.2, R33.2
- new net: J62.2 (Pin_2), R34.1
- new net: J69.2 (Pin_2), R39.1
- new net: J73.2 (Pin_2), R41.1
- new net: C11.1, J43.26, L9.2, R25.2, R26.2, R27.2
- new net: C14.1, J43.23, L12.2, R34.2, R35.2, R36.2
- new net: J43.28, J44.1 (1_1), J44.2 (1_2)
- new net: J52.2 (Pin_2), R29.1
- new net: J14.28, J44.3 (2_1), J44.4 (2_2)
- new net: J57.2 (Pin_2), R32.1
- new net: J48.2 (Pin_2), R27.1
- new net: J47.2 (Pin_2), R26.1
- new net: J68.2 (Pin_2), R38.1
- new net: J77.2 (Pin_2), R43.1
- new net: J56.2 (Pin_2), R31.1
- new net: J79.2 (Pin_2), R45.1
- new net: J63.2 (Pin_2), R35.1
- new net: J84.2 (Pin_2), R48.1
Other:
- moved on the sheet: C1, C2, C3, C4, C5, C6, C7, C8, J1, J10, J11, J12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

Commit message: Schematic Complete
Connections:
- net GND: now also C10.1, C9.2, J14.12, J43.12, J45.15 (8_1), J45.16 (8_2)
- net at C10.2: now also J14.01, J43.01, J45.3 (2_1), J45.4 (2_2)
- net at J43.14: now also J14.14, J45.13 (7_1), J45.14 (7_2)
- net at J43.15: now also J14.15, J45.11 (6_1), J45.12 (6_2)
- net at J43.16: now also J14.16, J45.10 (5_2), J45.9 (5_1)
- net at J43.17: now also J14.17, J45.7 (4_1), J45.8 (4_2)
- net at J43.18: now also J14.18, J45.5 (3_1), J45.6 (3_2)
- net at J43.27: now also C9.1, J14.27, J45.1 (1_1), J45.2 (1_2)
Other:
- moved on the sheet: C10, C9, J44
