File: measurementcircuit/measurementcircuit.kicad_pcb (KiCad board)
At the start: 4 copper layers, 174.5 x 220 mm, 150 parts, among them J1 Conn_01x02, J10 Conn_01x02, J11 Conn_01x02, J12 Conn_01x02, J13 2604-3102, J15 Conn_01x02, J16 Conn_01x02, J17 Conn_01x02, J18 2604-3102, J19 2604-3102, J2 Conn_01x02, J20 2604-3102, J21 Conn_01x02, J22 Conn_01x02, J23 Conn_01x02, J24 Conn_01x02, J25 Conn_01x02, J26 Conn_01x02, J27 Conn_01x02, J28 Conn_01x02, J29 Conn_01x02, J3 2604-3102, J30 Conn_01x02, J31 Conn_01x02, J32 Conn_01x02, J33 Conn_01x02, J34 Conn_01x02, J35 Conn_01x02, J36 Conn_01x02, J37 Conn_01x02, J38 Conn_01x02, J39 Conn_01x02, J4 2604-3102, J40 Conn_01x02, J41 Conn_01x02, J42 Conn_01x02, J47 Conn_01x02, J48 Conn_01x02, J49 Conn_01x02, J5 2604-3102, J51 Conn_01x02, J52 Conn_01x02, J53 Conn_01x02, J54 Conn_01x02, J56 Conn_01x02, J57 Conn_01x02, J58 Conn_01x02, J59 Conn_01x02, J6 2604-3102, J62 Conn_01x02, J63 Conn_01x02, J64 Conn_01x02, J65 Conn_01x02, J67 Conn_01x02, J68 Conn_01x02, J69 Conn_01x02, J7 2604-3102, J70 Conn_01x02, J72 Conn_01x02, J73 Conn_01x02, J74 Conn_01x02, J75 Conn_01x02, J77 Conn_01x02, J78 Conn_01x02, J79 Conn_01x02, J8 Conn_01x02, J80 Conn_01x02, J82 Conn_01x02, J83 Conn_01x02, J84 Conn_01x02, J9 Conn_01x02

Commit message: Add footprints, reassign footprints, change power supply connectors to new 2-pole style
Parts:
- added C10: C3216X7R1E475K160AC, 4.7uF_Bulk_Cap:CAP_3216_TDK, F.Cu at (53.9, 84.4)
- added C17: 10pF, 10pF_Capacitor_Custom:C_Disc_Radial_P5.90mm_W4.3mm_L11.4mm_Placeholder, F.Cu at (54.4, 96.4)
- added C19: CL10B104KB8NNNC, 0.1uF_Decoup_Cap:CAPC1608X90N, F.Cu at (138.7, 48.2)
- added C20: CL10B105KA8NNNC, 1uF_Local_Bulk_Cap:CAPC1608X90N, F.Cu at (138.7, 50.7)
- added C21: CL10B104KB8NNNC, 0.1uF_Decoup_Cap:CAPC1608X90N, F.Cu at (138.7, 53.1)
- added C22: CL10B105KA8NNNC, 1uF_Local_Bulk_Cap:CAPC1608X90N, F.Cu at (138.7, 55.6)
- added C23: C3216X7R1E475K160AC, 4.7uF_Bulk_Cap:CAP_3216_TDK, F.Cu at (53.9, 87.8)
- added C24: CL10B104KB8NNNC, 0.1uF_Decoup_Cap:CAPC1608X90N, F.Cu at (138.7, 58.1)
- added C25: CL10B105KA8NNNC, 1uF_Local_Bulk_Cap:CAPC1608X90N, F.Cu at (138.7, 60.6)
- added C26: C3216X7R1E475K160AC, 4.7uF_Bulk_Cap:CAP_3216_TDK, F.Cu at (53.9, 91.3)
- added C27: CL10B104KB8NNNC, 0.1uF_Decoup_Cap:CAPC1608X90N, F.Cu at (138.7, 63.1)
- added C28: CL10B105KA8NNNC, 1uF_Local_Bulk_Cap:CAPC1608X90N, F.Cu at (138.7, 65.5)
- added C9: C3216X7R1E475K160AC, 4.7uF_Bulk_Cap:CAP_3216_TDK, F.Cu at (53.9, 80.9)
- added J14: DILB28P-223TLF, DIP socket DILB28P_223TLF:AMPHENOL_DILB28P-223TLF, F.Cu at (107.1, 65.5)
- added J43: DILB28P-223TLF, DIP socket DILB28P_223TLF:AMPHENOL_DILB28P-223TLF, F.Cu at (127.0, 65.5)
- added J44: 2601-1102, 2_pole_term_block:CONN2_2601-1102_WAG, F.Cu at (55.9, 65.8)
- added J45: 2601-1108, 8_Pole_Terminal_Block:CONN8_2601-1108_WAG, F.Cu at (22.5, 65.8)
- added J46: 2601-1108, 8_Pole_Terminal_Block:CONN8_2601-1108_WAG, F.Cu at (22.5, 84.2)
- added J50: 2604-3102, 2_pole_term_block:CONN2_2601-1102_WAG, F.Cu at (-0.11, 43.0)
- added J55: 2604-3102, 2_pole_term_block:CONN2_2601-1102_WAG, F.Cu at (12.3, 43.0)
- added J60: 2601-1108, 8_Pole_Terminal_Block:CONN8_2601-1108_WAG, F.Cu at (22.5, 102.5)
- added J61: 2604-3102, 2_pole_term_block:CONN2_2601-1102_WAG, F.Cu at (24.6, 43.0)
- added J66: 2604-3102, 2_pole_term_block:CONN2_2601-1102_WAG, F.Cu at (37.0, 43.0)
- added J71: 2604-3102, 2_pole_term_block:CONN2_2601-1102_WAG, F.Cu at (49.4, 43.0)
- added J76: 2604-3102, 2_pole_term_block:CONN2_2601-1102_WAG, F.Cu at (61.7, 43.0)
- added J81: 2604-3102, 2_pole_term_block:CONN2_2601-1102_WAG, F.Cu at (74.1, 43.0)
- C1, C11, C12, C13, C14, C15, C16, C18, C2, C3, C4, C5, C6, C7, C8: footprint Capacitor_SMD:C_0805_2012Metric -> 10pF_Capacitor_Custom:C_Disc_Radial_P5.90mm_W4.3mm_L11.4mm_Placeholder
- J13: footprint WAGO_250-108/000-006_connector_BLUE.pretty:CONN8_250-108&slash_000-006_WAG -> 2_pole_term_block:CONN2_2601-1102_WAG
- J18, J19, J20, J3, J4, J5, J6, J7: footprint Wago - 2604-3302_2_pole_connector:CONN2_2604-3302_WAG -> 2_pole_term_block:CONN2_2601-1102_WAG
- L1, L10, L11, L12, L13, L14, L15, L16, L2, L3, L4, L5, L6, L7, L8, L9: footprint Inductor_SMD:L_0805_2012Metric -> 56uH_Inductor:INDAD1400W80L920D650
- R1, R10, R13, R16, R19, R22, R25, R28, R31, R34, R37, R4, R40, R43, R46, R7: footprint Resistor_THT:R_Axial_Power_L38.0mm_W9.0mm_P40.64mm -> 10Ohm Resistor:RS010_VIS
- R11, R14, R17, R2, R20, R23, R26, R29, R32, R35, R38, R41, R44, R47, R5, R8: footprint Resistor_THT:R_Axial_Power_L20.0mm_W6.4mm_P25.40mm -> 50Ohm_R:RES_CMF60_VIS
- R12, R15, R18, R21, R24, R27, R3, R30, R33, R36, R39, R42, R45, R48, R6, R9: footprint Resistor_THT:R_Axial_DIN0309_L9.0mm_D3.2mm_P5.08mm_Vertical -> 500Ohm_R:CMF65_VIS
- moved J20 9.03 mm to (-62.5, 127.5), turned to 90 degrees
- turned J18 to 90 degrees
- turned J19 to 90 degrees
- turned J3 to 90 degrees
- turned J4 to 90 degrees
- turned J5 to 90 degrees
- turned J6 to 90 degrees
- turned J7 to 90 degrees
Connections:
- C1 pad 1: Net-(J4-1_1) -> Net-(C1-Pad1)
- J4 pad 1: Net-(J4-1_1) -> Net-(J22-Pin_1)
- J4 pad 2: Net-(J4-1_1) -> Net-(J22-Pin_1)
- J9 pad 2: Net-(J4-1_1) -> Net-(J22-Pin_1)
- L2 pad 2: Net-(J4-1_1) -> Net-(C1-Pad1)
- R4 pad 2: Net-(J4-1_1) -> Net-(C1-Pad1)
- R5 pad 2: Net-(J4-1_1) -> Net-(C1-Pad1)
- R6 pad 2: Net-(J4-1_1) -> Net-(C1-Pad1)
Routing:
- net Net-(C1-Pad1): track 0.00 -> 199.6 mm, vias 0 -> 1
- net Net-(J13-1_1): track 0.00 -> 151.6 mm
- net Net-(C2-Pad1): track 284.3 -> 132.6 mm, vias 0 -> 1
- net Net-(C8-Pad1): track 212.3 -> 66.4 mm, vias 0 -> 1
- net GND: track 70.1 -> 216.0 mm, vias 24 -> 15
- net Net-(J22-Pin_1): track 272.5 -> 136.6 mm
- net Net-(J33-Pin_2): track 39.7 -> 172.9 mm
- net Net-(C6-Pad1): track 200.3 -> 67.1 mm, vias 0 -> 1
- net Net-(J4-1_1): track 63.6 -> 0.00 mm
- net Net-(J16-Pin_1): vias 0 -> 1
- net Net-(C7-Pad1): vias 0 -> 1
- net Net-(C5-Pad1): vias 0 -> 1
- net Net-(C4-Pad1): vias 0 -> 1
- net Net-(C3-Pad1): vias 0 -> 1

Commit message: PCB work, footing placement
Parts:
- J17, J45, J46, J60: moved to B.Cu
- moved C11 365.0 mm to (-305.6, -93.0)
- moved C13 362.5 mm to (-306.6, -71.5)
- moved C12 362.2 mm to (-305.1, -80.0)
- moved C14 361.8 mm to (-307.1, -62.0)
- moved C15 354.6 mm to (-301.6, -48.5)
- moved C16 354.0 mm to (-302.6, -35.0)
- moved C18 351.6 mm to (-300.6, -28.0)
- moved L9 337.0 mm to (-271.0, -97.0)
- moved L10 335.2 mm to (-271.0, -87.5)
- moved L14 330.9 mm to (-271.5, -55.5)
- moved L11 330.2 mm to (-270.5, -65.0)
- moved L15 330.1 mm to (-272.5, -43.0)
- moved L16 329.6 mm to (-273.5, -30.5)
- moved L12 324.1 mm to (-260.0, -80.5)
- moved L13 322.6 mm to (-260.0, -71.5)
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Routing:
- net Net-(J10-Pin_1): track 240.4 -> 0.00 mm
- net GND: track 216.0 -> 0.00 mm, vias 15 -> 0
- net Net-(C7-Pad1): track 203.5 -> 0.00 mm, vias 1 -> 0
- net Net-(C1-Pad1): track 199.6 -> 0.00 mm, vias 1 -> 0
- net Net-(C3-Pad1): track 193.5 -> 0.00 mm, vias 1 -> 0
- net Net-(C5-Pad1): track 188.9 -> 0.00 mm, vias 1 -> 0
- net Net-(J33-Pin_2): track 172.9 -> 0.00 mm
- net Net-(J13-1_1): track 151.6 -> 0.00 mm
- net Net-(J1-Pin_1): track 151.3 -> 0.00 mm
- net Net-(J46-8_1): track 0.00 -> 151.1 mm
- net Net-(J16-Pin_1): track 147.8 -> 0.00 mm, vias 1 -> 0
- net Net-(J22-Pin_1): track 136.6 -> 0.00 mm
- net Net-(J15-Pin_1): track 133.4 -> 0.00 mm
- net Net-(C2-Pad1): track 132.6 -> 0.00 mm, vias 1 -> 0
- net Net-(J10-Pin_2): track 123.4 -> 0.00 mm
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Other:
- board size 174.5 x 220 mm -> 250 x 275 mm

Commit message: Place Resistors, other footprint placements
Parts:
- C17, J13, J44, J50, J55, J61, J66, J71, J76, J81: moved to B.Cu
- moved R26 354.7 mm to (-153.4, 172.0)
- moved R25 336.4 mm to (-134.0, 180.5)
- moved R29 329.1 mm to (-153.4, 139.5)
- moved R27 324.9 mm to (-150.1, 162.0)
- moved C17 316.4 mm to (-199.5, -42.9), turned to -90 degrees
- moved R32 306.0 mm to (-153.4, 105.5)
- moved R30 298.6 mm to (-150.1, 127.5)
- moved R28 290.1 mm to (-133.5, 148.5)
- moved R35 286.9 mm to (-153.4, 71.0)
- moved C11 276.5 mm to (-200.0, 162.6), turned to -90 degrees
- moved R33 275.4 mm to (-150.1, 93.0)
- moved R38 273.3 mm to (-153.4, 37.0)
- moved L9 272.1 mm to (-216.0, 169.5), turned to 90 degrees
- moved R47 270.7 mm to (-153.9, -66.0)
- moved R41 265.6 mm to (-153.4, 2.50)
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
Commit message: Major PCB work, Ready for review
Still need to reassign 3D models
Parts:
- moved J47 300.2 mm to (-133.5, 172.0), turned to 90 degrees
- moved J48 297.3 mm to (-141.5, 162.0), turned to 90 degrees
- moved J51 266.8 mm to (-123.0, 148.5), turned to 90 degrees
- moved J52 266.3 mm to (-133.0, 139.5), turned to 90 degrees
- moved J53 263.5 mm to (-141.5, 127.5), turned to 90 degrees
- moved J79 258.0 mm to (-142.5, -44.0), turned to 90 degrees
- moved J57 255.7 mm to (-133.5, 105.5), turned to 90 degrees
- moved J58 254.2 mm to (-141.5, 93.0), turned to 90 degrees
- moved J56 253.8 mm to (-123.0, 114.0), turned to 90 degrees
- moved J49 253.1 mm to (-103.0, 146.5), turned to 0 degrees
- moved J64 251.9 mm to (-141.5, 59.0), turned to 90 degrees
- moved J63 251.1 mm to (-133.5, 71.0), turned to 90 degrees
- moved J78 250.5 mm to (-133.5, -31.0), turned to 90 degrees
- moved C19 250.0 mm to (-76.0, -2.78), turned to -90 degrees
- moved C24 244.7 mm to (-76.0, 61.2), turned to -90 degrees
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Routing:
- net Net-(C11-Pad1): track 0.00 -> 423.6 mm
- net Net-(C12-Pad1): track 0.00 -> 390.4 mm
- net Net-(C18-Pad1): track 0.00 -> 366.1 mm
- net Net-(C17-Pad1): track 0.00 -> 363.2 mm
- net Net-(C16-Pad1): track 0.00 -> 350.6 mm
- net Net-(C13-Pad1): track 0.00 -> 344.5 mm
- net Net-(C2-Pad1): track 0.00 -> 296.1 mm
- net Net-(C14-Pad1): track 0.00 -> 295.8 mm
- net Net-(J75-Pin_2): track 0.00 -> 287.9 mm
- net Net-(J80-Pin_2): track 0.00 -> 278.6 mm
- net Net-(C8-Pad1): track 0.00 -> 274.8 mm
- net Net-(J70-Pin_2): track 0.00 -> 268.2 mm
- net Net-(C7-Pad1): track 0.00 -> 255.7 mm
- net Net-(J1-Pin_1): track 0.00 -> 245.5 mm
- net Net-(C6-Pad1): track 0.00 -> 243.3 mm
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Other:
- board size 250 x 275 mm -> 225 x 275 mm

Commit message: Finish PCB, Schematic and PCB ready for review
Other:
- board text added: "~ Plasma Frontiers ~ SDSU Senior Design 2025-2026 Daniel Self, Son Huynh, Ulises Urbina, Jimin Chae, & Clayton Alvarez."
